File: KICAD diseño/PLC DISEÑO/INPUT_NPN.kicad_sch (KiCad schematic)
At the start: 0 parts

Commit message: Actualizacion
Parts:
- added D2: DL4007, PCM_Diode_SMD_AKL:D_MELF, symbol PCM_Diode_AKL:DL4007
- added OC1: LTV-357T, PCM_Package_SO_AKL:SO-4_4.4x3.9mm_P2.54mm, symbol PCM_Optocoupler_AKL:LTV-357T
- added R4, R5: R_0603, PCM_Resistor_SMD_AKL:R_0603_1608Metric, symbol PCM_Resistor_US_AKL:R_0603
Connections:
- new net: D2.1 (K), OC1.1, R4.2
- new net +3.3V: R5.1
- new net GND: OC1.3
- new net NPN_in +: R4.1
- new net NPN_in -: D2.2 (A), OC1.2
- new net NPN_input: OC1.4, R5.2
