File: KICAD diseño/PLC DISEÑO/Powersuply.kicad_sch (KiCad schematic)
At the start: 5 parts, among them U2 AP63203WU

Commit message: Update
Parts:
- added C5, C6: 22uF, PCM_Capacitor_SMD_AKL:C_0603_1608Metric, symbol PCM_Capacitor_AKL:C_0603
- added R2, R3: 22k, PCM_Resistor_SMD_AKL:R_0603_1608Metric, symbol PCM_Resistor_US_AKL:R_0603
- C3, C4: value C_0603 -> 100pF
Connections:
- net +3.3V: now also C4.1, L1.2, C5.1, C6.1, R2.1
- net VCC: now also C2.1, U2.2 (EN), U2.3 (IN)
- net at U2.1 (FB): now also C4.2, R2.2, R3.1
- net GND: now reaches U2.4 (GND)
- net GND: now also C5.2, C6.2, R3.2
- net at U2.5 (SW): now also C3.2, L1.1
- net at U2.6 (BST): now also C3.1
Other:
- moved on the sheet: C2, C3, C4, L1, U2

Commit message: Actualizacion
Connections:
- net GND: now also C2.2
Other:
- moved on the sheet: C3
Changed lines of the file:
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@@
+	)
+	(junction
+		(at 142.24 41.91)
+		(diameter 0)
+		(color 0 0 0 0)
 	)
 	(junction
@@
 	(wire
 		(pts
-			(xy 137.16 38.1) (xy 137.16 41.91)
+			(xy 142.24 41.91) (xy 142.24 50.8)
 		)
 		(stroke
@@
 	(wire
 		(pts
+			(xy 137.16 41.91) (xy 137.16 38.1)
+		)
+		(stroke
+			(width 0)
+			(type default)
+		)
+	)
+	(wire
+		(pts
 			(xy 151.13 30.48) (xy 151.13 27.94)
 		)
@@
 	(wire
 		(pts
-			(xy 124.46 26.67) (xy 124.46 27.94)
+			(xy 124.46 19.05) (xy 124.46 27.94)
 		)
 		(stroke
@@
 	(wire
 		(pts
+			(xy 142.24 41.91) (xy 137.16 41.91)
+		)
+		(stroke
+			(width 0)
+			(type default)
+		)
+	)
+	(wire
+		(pts
 			(xy 151.13 38.1) (xy 151.13 41.91)
 		)
@@
 	(wire
 		(pts
-			(xy 85.09 35.56) (xy 85.09 20.32)
-		)
-		(stroke
-			(width 0)
-			(type default)
-		)
-	)
-	(wire
-		(pts
-			(xy 92.71 20.32) (xy 92.71 27.94)
+			(xy 92.71 35.56) (xy 92.71 27.94)
+		)
+		(stroke
+			(width 0)
+			(type default)
+		)
+	)
+	(wire
+		(pts
+			(xy 151.13 41.91) (xy 142.24 41.91)
 		)
 		(stroke
@@
 		(pts
 			(xy 30.48 33.02) (xy 30.48 38.1)
+		)
+		(stroke
+			(width 0)
+			(type default)
+		)
+	)
+	(wire
+		(pts
+			(xy 30.48 45.72) (xy 30.48 48.26)
 		)
 		(stroke
@@
 	(symbol
 		(lib_id "power:GND")
+		(at 30.48 48.26 0)
+		(unit 1)
+		(exclude_from_sim no)
+		(in_bom yes)
+		(on_board yes)
+		(dnp no)
+		(fields_autoplaced yes)
+		(property "Reference" "#PWR017"
+			(at 30.48 54.61 0)
+			(effects
+				(font
+					(size 1.27 1.27)
+				)
+				(hide yes)
+			)
+		)
+		(property "Value" "GND"
+			(at 30.48 53.34 0)
+			(effects
+				(font
+					(size 1.27 1.27)
+				)
+			)
+		)
+		(property "Footprint" ""
+			(at 30.48 48.26 0)
+			(effects
+				(font
+					(size 1.27 1.27)
+				)
+				(hide yes)
+			)
+		)
+		(property "Datasheet" ""
+			(at 30.48 48.26 0)
+			(effects
+				(font
+					(size 1.27 1.27)
+				)
+				(hide yes)
+			)
+		)
+		(property "Description" "Power symbol creates a global label with name \"GND\" , ground"
+			(at 30.48 48.26 0)
+			(effects
+				(font
+					(size 1.27 1.27)
+				)
+				(hide yes)
+			)
+		)
+		(pin "1"
+		)
+		(instances
+			(project "PLC DISEÑO"
+				(path "/3591d221-fcc3-4bcd-9e55-dff6b841bafc/6cae9003-6268-4873-a546-b84fa61fb294/46341553-5d04-4231-997f-c9f7c3a4d636"
+					(reference "#PWR017")
+					(unit 1)
+				)
+			)
+		)
+	)
+	(symbol
+		(lib_id "power:GND")
 		(at 124.46 59.69 0)
 		(unit 1)
@@
 	(symbol
 		(lib_id "PCM_Capacitor_AKL:C_0603")
-		(at 88.9 20.32 90)
+		(at 88.9 35.56 90)
 		(unit 1)
 		(exclude_from_sim no)
@@
 		(fields_autoplaced yes)
 		(property "Reference" "C3"
-			(at 88.9 12.7 90)
+			(at 88.9 27.94 90)
 			(effects
 				(font
@@
 		)
 		(property "Value" "100pF"
-			(at 88.9 15.24 90)
+			(at 88.9 30.48 90)
 			(effects
 				(font
@@
 		)
 		(property "Footprint" "PCM_Capacitor_SMD_AKL:C_0603_1608Metric"
-			(at 92.71 19.3548 0)
+			(at 92.71 34.5948 0)
 			(effects
 				(font
@@
 		)
 		(property "Datasheet" "~"
-			(at 88.9 20.32 0)
+			(at 88.9 35.56 0)
 			(effects
 				(font
@@
 		)
 		(property "Description" "SMD 0603 MLCC capacitor, Alternate KiCad Library"
-			(at 88.9 20.32 0)
+			(at 88.9 35.56 0)
 			(effects
 				(font
@@
 	(symbol
 		(lib_id "power:GND")
-		(at 137.16 41.91 0)
+		(at 142.24 50.8 0)
 		(unit 1)
 		(exclude_from_sim no)
@@
 		(fields_autoplaced yes)
 		(property "Reference" "#PWR010"
-			(at 137.16 48.26 0)
+			(at 142.24 57.15 0)
 			(effects
 				(font
@@
 		)
 		(property "Value" "GND"
-			(at 137.16 46.99 0)
+			(at 142.24 55.88 0)
 			(effects
 				(font
@@
 		)
 		(property "Footprint" ""
-			(at 137.16 41.91 0)
+			(at 142.24 50.8 0)
 			(effects
 				(font
@@
 		)
 		(property "Datasheet" ""
-			(at 137.16 41.91 0)
+			(at 142.24 50.8 0)
 			(effects
 				(font
@@
 		)
 		(property "Description" "Power symbol creates a global label with name \"GND\" , ground"
-			(at 137.16 41.91 0)
+			(at 142.24 50.8 0)
 			(effects
 				(font
@@
 	(symbol
 		(lib_id "power:+3.3V")
-		(at 124.46 26.67 0)
+		(at 124.46 19.05 0)
 		(unit 1)
 		(exclude_from_sim no)
@@
 		(fields_autoplaced yes)
 		(property "Reference" "#PWR04"
-			(at 124.46 30.48 0)
+			(at 124.46 22.86 0)
 			(effects
 				(font
@@
 		)
 		(property "Value" "+3.3V"
-			(at 124.46 21.59 0)
+			(at 124.46 13.97 0)
 			(effects
 				(font
@@
 		)
 		(property "Footprint" ""
-			(at 124.46 26.67 0)
+			(at 124.46 19.05 0)
 			(effects
 				(font
@@
 		)
 		(property "Datasheet" ""
-			(at 124.46 26.67 0)
+			(at 124.46 19.05 0)
 			(effects
 				(font
@@
 		)
 		(property "Description" "Power symbol creates a global label with name \"+3.3V\""
-			(at 124.46 26.67 0)
+			(at 124.46 19.05 0)
 			(effects
 				(font
@@
 					(unit 1)
 				)
-			)
-		)
-	)
-	(symbol
-		(lib_id "power:GND")
-		(at 151.13 41.91 0)
-		(unit 1)
-		(exclude_from_sim no)
-		(in_bom yes)
-		(on_board yes)
-		(dnp no)
-		(fields_autoplaced yes)
-		(property "Reference" "#PWR014"
-			(at 151.13 48.26 0)
-			(effects
-				(font
-					(size 1.27 1.27)
-				)
-				(hide yes)
-			)
-		)
-		(property "Value" "GND"
-			(at 151.13 46.99 0)
-			(effects
-				(font
-					(size 1.27 1.27)
-				)
-			)
-		)
-		(property "Footprint" ""
-			(at 151.13 41.91 0)
-			(effects
-				(font
-					(size 1.27 1.27)
-				)
-				(hide yes)
-			)
-		)
-		(property "Datasheet" ""
-			(at 151.13 41.91 0)
-			(effects
-				(font
-					(size 1.27 1.27)
-				)
-				(hide yes)
-			)
-		)
-		(property "Description" "Power symbol creates a global label with name \"GND\" , ground"
-			(at 151.13 41.91 0)
-			(effects
-				(font
-					(size 1.27 1.27)
-				)
-				(hide yes)
-			)
-		)
-		(pin "1"
-		)
-		(instances
-			(project ""
-				(path "/3591d221-fcc3-4bcd-9e55-dff6b841bafc/6cae9003-6268-4873-a546-b84fa61fb294/46341553-5d04-4231-997f-c9f7c3a4d636"
-					(reference "#PWR014")
-					(unit 1)
-				)
