File: KICAD diseño/PLC DISEÑO/DRIVER_RS485.kicad_sch (KiCad schematic)
At the start: 0 parts

Commit message: Update
Parts:
- added C7: ~, Library:C2992406, symbol PCM_SL_Connectors:C2992406
Changed lines of the file:
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@@
+		)
+	)
+	(symbol
+		(lib_id "PCM_SL_Connectors:C2992406")
+		(at 92.71 49.53 0)
+		(unit 1)
+		(exclude_from_sim no)
+		(in_bom yes)
+		(on_board yes)
+		(dnp no)
+		(property "Reference" "C7"
+			(at 122.682 68.58 0)
+			(effects
+				(font
+					(size 1.27 1.27)
+				)
+			)
+		)
+		(property "Value" "~"
+			(at 122.555 68.58 0)
+			(effects
+				(font
+					(size 1.27 1.27)
+				)
+			)
+		)
+		(property "Footprint" "Library:C2992406"
+			(at 121.92 67.31 0)
+			(effects
+				(font
+					(size 1.27 1.27)
+				)
+				(hide yes)
+			)
+		)
+		(property "Datasheet" ""
+			(at 121.92 67.31 0)
+			(effects
+				(font
+					(size 1.27 1.27)
+				)
+				(hide yes)
+			)
+		)
+		(property "Description" ""
+			(at 121.92 67.31 0)
+			(effects
+				(font
+					(size 1.27 1.27)
+				)
+				(hide yes)
+			)
+		)
+		(pin "5"
+		)
+		(pin "8"
+		)
+		(pin "8"
+		)
+		(pin "10"
+		)
+		(pin "3"
+		)
+		(pin "1"
+		)
+		(pin "2"
+		)
+		(pin "4"
+		)
+		(instances
+			(project ""
+				(path "/3591d221-fcc3-4bcd-9e55-dff6b841bafc/6cae9003-6268-4873-a546-b84fa61fb294/9035043c-eb7b-4ac1-ab01-e544e69f90aa"
+					(reference "C7")
+					(unit 1)
+				)
+			)
 		)
 	)

Commit message: Actualizacion
Parts:
- added C8: C_0603, PCM_Capacitor_SMD_AKL:C_0603_1608Metric, symbol PCM_Capacitor_AKL:C_0603
- added D1: SM712, PCM_Package_TO_SOT_SMD_AKL:SOT-23, symbol PCM_Diode_TVS_AKL:SM712
Connections:
- net RS485-A: now also C7.9 (A)
- net RS485-B: now also C7.8 (B)
- net UART_IN: now also C7.3 (TXD)
- net UART_OUT: now also C7.4 (RXD)
- net +3.3V: now reaches C7.1 (VCC)
- net +3.3V: now also C8.1, D1.2 (A2)
- net at C7.2 (GND): now also C8.2, D1.1 (A1)
- net GPIO control: now reaches C7.5 (CON)
- new net GND: D1.3 (Com)

Commit message: Actualizacion estoy cansado jefe :)
Changed lines of the file:
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@@
 	(wire
 		(pts
-			(xy 114.3 73.66) (xy 101.6 73.66)
+			(xy 114.3 73.66) (xy 100.33 73.66)
 		)
 		(stroke
@@
 	(wire
 		(pts
-			(xy 101.6 80.01) (xy 95.25 80.01)
+			(xy 100.33 80.01) (xy 95.25 80.01)
 		)
 		(stroke
@@
 	(wire
 		(pts
-			(xy 101.6 73.66) (xy 101.6 80.01)
+			(xy 100.33 73.66) (xy 100.33 80.01)
 		)
 		(stroke
