File: KICAD diseño/PLC DISEÑO/INPUT_PNP.kicad_sch (KiCad schematic)
At the start: 0 parts

Commit message: Actualizacion
Parts:
- added D3: DL4007, PCM_Diode_SMD_AKL:D_MELF, symbol PCM_Diode_AKL:DL4007
- added OC2: LTV-357T, PCM_Package_SO_AKL:SO-4_4.4x3.9mm_P2.54mm, symbol PCM_Optocoupler_AKL:LTV-357T
- added R6, R7: R_0603, PCM_Resistor_SMD_AKL:R_0603_1608Metric, symbol PCM_Resistor_US_AKL:R_0603
Connections:
- new net: D3.1 (K), OC2.1, R6.2
- new net +3.3V: OC2.4
- new net GND: R7.1
- new net NPN_in +: R6.1
- new net PNP_in -: D3.2 (A), OC2.2
- new net PNP_input: OC2.3, R7.2

Commit message: Actualizacion estoy cansado jefe :)
Parts:
- added D5: DL4007, PCM_Diode_SMD_AKL:D_MELF, symbol PCM_Diode_AKL:DL4007
- added OC4: LTV-357T, PCM_Package_SO_AKL:SO-4_4.4x3.9mm_P2.54mm, symbol PCM_Optocoupler_AKL:LTV-357T
- added R10, R11: R_0603, PCM_Resistor_SMD_AKL:R_0603_1608Metric, symbol PCM_Resistor_US_AKL:R_0603
Connections:
- net PNP_in - is gone; now on net GND: D3.2 (A), OC2.2
- net +3.3V: now also OC4.4
- net GND: now also D5.2 (A), OC4.2, R11.1
- net NPN_in + renamed PNP_in + 1
- net PNP_input renamed PNP_input_1
- new net: D5.1 (K), OC4.1, R10.2
- new net PNP_in + 2: R10.1
- new net PNP_input_2: OC4.3, R11.2
