File: KICAD diseño/PLC DISEÑO/Modulo420.kicad_sch (KiCad schematic)
At the start: 8 parts

Commit message: Actualizacion estoy cansado jefe :)
Parts:
- removed D2, D4: DL4007, PCM_Diode_SMD_AKL:D_MELF, symbol PCM_Diode_AKL:DL4007
- removed OC1, OC3: LTV-357T, PCM_Package_SO_AKL:SO-4_4.4x3.9mm_P2.54mm, symbol PCM_Optocoupler_AKL:LTV-357T
- removed R4, R5, R8, R9: R_0603, PCM_Resistor_SMD_AKL:R_0603_1608Metric, symbol PCM_Resistor_US_AKL:R_0603
- added C10, C9: C_0603, PCM_Capacitor_SMD_AKL:C_0603_1608Metric, symbol PCM_Capacitor_AKL:C_0603
- added R12, R13, R14: R_0603, PCM_Resistor_SMD_AKL:R_0603_1608Metric, symbol PCM_Resistor_US_AKL:R_0603
- added U4: GP8303-TC50-EW, EasyEDA:ESOP-10_L4.9-W3.9-P1.00-LS6.1-BL-EP, symbol Cris:GP8303-TC50-EW
Connections:
- net +3.3V: now also R12.1, R13.1
- net GND: now also C10.1, C9.2, R14.2, U4.3 (A0), U4.4 (A1), U4.6 (GND), U4.9 (A2)
- new net: C9.1, R14.1, U4.7 (SET)
- new net: C10.2, U4.10 (V5V)
- new net ASLK: R13.2, U4.1 (SLCK)
- new net SDA: R12.2, U4.2 (SDA)
- new net VCC: U4.5 (VCC)
- new net out_420mA: U4.8 (IOUT)
