File: KICAD diseño/PLC DISEÑO/PLC DISEÑO.kicad_sch (KiCad schematic)
At the start: 11 parts, among them J1 Screw_Terminal_01x02, J10 Screw_Terminal_3_P5.00mm, J11 Screw_Terminal_2_P5.00mm, J14 Screw_Terminal_6_P5.00mm, J2 Screw_Terminal_4_P5.00mm, J4 Screw_Terminal_2_P5.00mm, J6 Screw_Terminal_3_P5.00mm, J7 Screw_Terminal_2_P5.00mm, J8 Screw_Terminal_2_P5.00mm, J9 Screw_Terminal_4_P5.00mm

Commit message: Update
Parts:
- removed J1: Screw_Terminal_01x02, symbol Connector:Screw_Terminal_01x02
- removed J11: Screw_Terminal_2_P5.00mm, TerminalBlock_Phoenix:TerminalBlock_Phoenix_PT-1,5-2-5.0-H_1x02_P5.00mm_Horizontal, symbol PCM_SL_Screw_Terminal:Screw_Terminal_2_P5.00mm
- added J1, J3: Screw_Terminal_2_P5.00mm, TerminalBlock_Phoenix:TerminalBlock_Phoenix_PT-1,5-2-5.0-H_1x02_P5.00mm_Horizontal, symbol PCM_SL_Screw_Terminal:Screw_Terminal_2_P5.00mm
- renumbered WIFI-BT to WIFI-BT1
Connections:
- net BOARD_NIRVARA/RUN/STOP: now also J3.1
- net GND: now also J1.2, J3.2
- net VCC: now also J1.1

Commit message: Actualizacion estoy cansado jefe :)
Changed lines of the file:
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@@
 	(text "Entrada Stop\n"
 		(exclude_from_sim no)
-		(at 83.82 135.89 0)
+		(at 83.312 135.89 0)
 		(effects
 			(font

Commit message: Nirvara actualization :>
Parts:
- added J5: Screw_Terminal_4_P5.00mm, TerminalBlock_Phoenix:TerminalBlock_Phoenix_PT-1,5-4-5.0-H_1x04_P5.00mm_Horizontal, symbol PCM_SL_Screw_Terminal:Screw_Terminal_4_P5.00mm
Connections:
- net BOARD_NIRVARA/RFL1_NC renamed BOARD_NIRVARA/RLY1_NC
- net BOARD_NIRVARA/RFL2_NC renamed BOARD_NIRVARA/RLY2_NC
- new net BOARD_NIRVARA/in + 1: J5.1
- new net BOARD_NIRVARA/in + 2: J5.3
- new net BOARD_NIRVARA/in - 1: J5.2
- new net BOARD_NIRVARA/in - 2: J5.4
Other:
- sheet BOARD_NIRVARA ports: added RLY1_NC, RLY2_NC, in + 1, in + 2, in - 1, in - 2; removed RFL1_NC, RFL2_NC
Changed lines of the file:
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@@
+	(wire
+		(pts
+			(xy 100.33 123.19) (xy 102.87 123.19)
+		)
+		(stroke
+			(width 0)
+			(type default)
+		)
+	)
 	(wire
 		(pts
@@
 	(wire
 		(pts
+			(xy 100.33 128.27) (xy 102.87 128.27)
+		)
+		(stroke
+			(width 0)
+			(type default)
+		)
+	)
+	(wire
+		(pts
+			(xy 100.33 125.73) (xy 102.87 125.73)
+		)
+		(stroke
+			(width 0)
+			(type default)
+		)
+	)
+	(wire
+		(pts
 			(xy 99.06 135.89) (xy 102.87 135.89)
+		)
+		(stroke
+			(width 0)
+			(type default)
+		)
+	)
+	(wire
+		(pts
+			(xy 100.33 130.81) (xy 102.87 130.81)
 		)
 		(stroke
@@
 	)
 	(symbol
+		(lib_id "PCM_SL_Screw_Terminal:Screw_Terminal_4_P5.00mm")
+		(at 96.52 127 0)
+		(mirror y)
+		(unit 1)
+		(exclude_from_sim no)
+		(in_bom yes)
+		(on_board yes)
+		(dnp no)
+		(property "Reference" "J5"
+			(at 95.885 134.62 0)
+			(effects
+				(font
+					(size 1.27 1.27)
+				)
+			)
+		)
+		(property "Value" "Screw_Terminal_4_P5.00mm"
+			(at 92.71 128.2699 0)
+			(effects
+				(font
+					(size 1.27 1.27)
+				)
+				(justify left)
+				(hide yes)
+			)
+		)
+		(property "Footprint" "TerminalBlock_Phoenix:TerminalBlock_Phoenix_PT-1,5-4-5.0-H_1x04_P5.00mm_Horizontal"
+			(at 96.52 135.89 0)
+			(effects
+				(font
+					(size 1.27 1.27)
+				)
+				(hide yes)
+			)
+		)
+		(property "Datasheet" ""
+			(at 96.52 124.46 0)
+			(effects
+				(font
+					(size 1.27 1.27)
+				)
+				(hide yes)
+			)
+		)
+		(property "Description" ""
+			(at 96.52 127 0)
+			(effects
+				(font
+					(size 1.27 1.27)
+				)
+				(hide yes)
+			)
+		)
+		(pin "3"
+		)
+		(pin "2"
+		)
+		(pin "4"
+		)
+		(pin "1"
+		)
+		(instances
+			(project "PLC DISEÑO"
+				(path "/3591d221-fcc3-4bcd-9e55-dff6b841bafc"
+					(reference "J5")
+					(unit 1)
+				)
+			)
+		)
+	)
+	(symbol
 		(lib_id "power:GND")
 		(at 154.94 95.25 0)
@@
 			)
 		)
-		(pin "AOUT_420_1" input
+		(pin "AOUT_420_1" output
 			(at 151.13 88.9 0)
 			(effects
@@
 			)
 		)
-		(pin "AOUT_010_1" input
+		(pin "AOUT_010_1" output
 			(at 151.13 86.36 0)
 			(effects
@@
 			)
 		)
-		(pin "RFL2_NC" output
-			(at 151.13 134.62 0)
-			(effects
-				(font
-					(size 1.27 1.27)
-				)
-				(justify right)
-			)
-		)
-		(pin "RFL1_NC" output
-			(at 151.13 127 0)
-			(effects
-				(font
-					(size 1.27 1.27)
-				)
-				(justify right)
-			)
-		)
 		(pin "RLY1_NO" output
 			(at 151.13 132.08 0)
@@
 			)
 		)
+		(pin "RLY2_NC" output
+			(at 151.13 134.62 0)
+			(effects
+				(font
+					(size 1.27 1.27)
+				)
+				(justify right)
+			)
+		)
+		(pin "RLY1_NC" output
+			(at 151.13 127 0)
+			(effects
+				(font
+					(size 1.27 1.27)
+				)
+				(justify right)
+			)
+		)
+		(pin "in + 1" input
+			(at 102.87 123.19 180)
+			(effects
+				(font
+					(size 1.27 1.27)
+				)
+				(justify left)
+			)
+		)
+		(pin "in - 2" input
+			(at 102.87 130.81 180)
+			(effects
+				(font
+					(size 1.27 1.27)
+				)
+				(justify left)
+			)
+		)
+		(pin "in - 1" input
+			(at 102.87 125.73 180)
+			(effects
+				(font
+					(size 1.27 1.27)
+				)
+				(justify left)
+			)
+		)
+		(pin "in + 2" input
+			(at 102.87 128.27 180)
+			(effects
+				(font
+					(size 1.27 1.27)
+				)
+				(justify left)
+			)
+		)
