File: KICAD diseño/PLC DISEÑO/untitled.kicad_sch (KiCad schematic)
At the start: 3 parts, among them U1 ESP32-S3-WROOM-1

Commit message: Actualizacion
Other:
- removed sheet OUTPUT_NPN
- removed sheet OUTPUT_PNP
- added sheet Realy (untitled2.kicad_sch)
- sheet DRIVER_RS485 ports: added GPIO control; removed none
- sheet INPUT_NPN ports: added NPN_in +, NPN_in -, NPN_input; removed none
- sheet INPUT_PNP ports: added NPN_in +, PNP_in -, PNP_input; removed none

Commit message: Actualizacion estoy cansado jefe :)
Parts:
- added R18: R_0603, PCM_Resistor_SMD_AKL:R_0603_1608Metric, symbol PCM_Resistor_US_AKL:R_0603
- U1: footprint PCM_Espressif:ESP32-S3-WROOM-1 -> ESP32-S3-WROM-1:ESP32-S3-WROOM-1
Connections:
- net +3.3V: now also R18.1
- net RUN/STOP: now also U1.29 (SPIIO7/GPIO36/FSPICLK/SUBSPICLK), R18.2
- net Realy/RLY_1: now also U1.5 (GPIO5/TOUCH5/ADC1_CH4)
- net Realy/RLY_2: now also U1.6 (GPIO6/TOUCH6/ADC1_CH5)
- net Modulo_out_420/SDA: now reaches U1.12 (GPIO8/TOUCH8/ADC1_CH7/SUBSPICS1)
- net INPUT_PNP/PNP_input_1: now reaches U1.15 (GPIO3/TOUCH3/ADC1_CH2)
- net 34_v/0_32Vin: now reaches U1.16 (GPIO46)
- net Modulo_010/SDA: now reaches U1.17 (GPIO9/TOUCH9/ADC1_CH8/FSPIHD/SUBSPIHD)
- net Modulo_010/SCLK: now reaches U1.18 (GPIO10/TOUCH10/ADC1_CH9/FSPICS0/FSPIIO4/SUBSPICS0)
- net INPUT_NPN/NPN_input_2: now reaches U1.38 (GPIO2/TOUCH2/ADC1_CH1)
- net INPUT_NPN/NPN_input_1: now reaches U1.39 (GPIO1/TOUCH1/ADC1_CH0)
- net INPUT_PNP/PNP_input_2: now reaches U1.4 (GPIO4/TOUCH4/ADC1_CH3)
- net Modulo_out_420/ASLK: now reaches U1.7 (GPIO7/TOUCH7/ADC1_CH6)
Other:
- added sheet 34_v (salida34.kicad_sch)
- added sheet Modulo_010 (Modulo010.kicad_sch)
- added sheet Modulo_out_420 (Modulo420.kicad_sch)
- sheet INPUT_NPN ports: added NPN_in + 1, NPN_in + 2, NPN_input_1, NPN_input_2; removed NPN_in +, NPN_in -, NPN_input
- sheet INPUT_PNP ports: added PNP_in + 1, PNP_in + 2, PNP_input_1, PNP_input_2; removed NPN_in +, PNP_in -, PNP_input
- moved on the sheet: C1, R1, U1

Commit message: Nirvara actualization :>
Connections:
- net 34_v/0_32Vin: now also U1.19 (GPIO11/TOUCH11/ADC2_CH0/FSPID/FSPIIO5/SUBSPID); no longer U1.16 (GPIO46)
- net Modulo_in/input_1: now reaches U1.26 (GPIO45)
- net 420_IN/420_in: now reaches U1.27 (GPIO0/BOOT)
- new net Modulo_in/input_2: U1.16 (GPIO46)
Other:
- added sheet 420_IN (entrada420.kicad_sch)
- added sheet Modulo_in (moduloin.kicad_sch)

Commit message: Actualizacion 20 :[
Connections:
- net 34_v/0_32Vin: now also U1.11 (GPIO18/U1RXD/ADC2_CH7/CLK_OUT3); no longer U1.19 (GPIO11/TOUCH11/ADC2_CH0/FSPID/FSPIIO5/SUBSPID)
- net 420_IN/420_in: now also U1.23 (GPIO21); no longer U1.27 (GPIO0/BOOT)
- net DRIVER_RS485/UART_IN: now also U1.21 (GPIO13/TOUCH13/ADC2_CH2/FSPIQ/FSPIIO7/SUBSPIQ); no longer U1.37 (U0TXD/GPIO43/CLK_OUT1)
- net DRIVER_RS485/UART_OUT: now also U1.22 (GPIO14/TOUCH14/ADC2_CH3/FSPIWP/FSPIDQS/SUBSPIWP); no longer U1.36 (U0RXD/GPIO44/CLK_OUT2)
- net INPUT_NPN/NPN_input_1: now also U1.5 (GPIO5/TOUCH5/ADC1_CH4); no longer U1.39 (GPIO1/TOUCH1/ADC1_CH0)
- net INPUT_NPN/NPN_input_2: now also U1.6 (GPIO6/TOUCH6/ADC1_CH5); no longer U1.38 (GPIO2/TOUCH2/ADC1_CH1)
- net INPUT_PNP/PNP_input_1: now also U1.7 (GPIO7/TOUCH7/ADC1_CH6); no longer U1.15 (GPIO3/TOUCH3/ADC1_CH2)
- net INPUT_PNP/PNP_input_2: now also U1.12 (GPIO8/TOUCH8/ADC1_CH7/SUBSPICS1); no longer U1.4 (GPIO4/TOUCH4/ADC1_CH3)
- net Modulo_in/input_1: now also U1.37 (U0TXD/GPIO43/CLK_OUT1); no longer U1.26 (GPIO45)
- net Modulo_in/input_2: now also U1.36 (U0RXD/GPIO44/CLK_OUT2); no longer U1.16 (GPIO46)
- net Modulo_out_420/ASLK: now also U1.19 (GPIO11/TOUCH11/ADC2_CH0/FSPID/FSPIIO5/SUBSPID); no longer U1.7 (GPIO7/TOUCH7/ADC1_CH6)
- net Modulo_out_420/SDA: now also U1.20 (GPIO12/TOUCH12/ADC2_CH1/FSPICLK/FSPIIO6/SUBSPICLK); no longer U1.12 (GPIO8/TOUCH8/ADC1_CH7/SUBSPICS1)
- net Realy/RLY_1: now also U1.14 (GPIO20/U1CTS/ADC2_CH9/CLK_OUT1/USB_D+); no longer U1.5 (GPIO5/TOUCH5/ADC1_CH4)
- net Realy/RLY_2: now also U1.13 (GPIO19/U1RTS/ADC2_CH8/CLK_OUT2/USB_D-); no longer U1.6 (GPIO6/TOUCH6/ADC1_CH5)
- net 0.10Vin/0-10V: now reaches U1.10 (GPIO17/U1TXD/ADC2_CH6)
- new net Out_NPN/NPN-1: U1.39 (GPIO1/TOUCH1/ADC1_CH0)
- new net Out_NPN/NPN-2: U1.38 (GPIO2/TOUCH2/ADC1_CH1)
- new net Out_PNP/PNP-1: U1.15 (GPIO3/TOUCH3/ADC1_CH2)
- new net Out_PNP/PNP-2: U1.4 (GPIO4/TOUCH4/ADC1_CH3)
Other:
- added sheet 0.10Vin (vin.kicad_sch)
- added sheet Out_NPN (out.kicad_sch)
- added sheet Out_PNP (Outpnp.kicad_sch)
- moved on the sheet: C1, R1, R18, U1
