File: KICAD diseño/PLC DISEÑO/untitled2.kicad_sch (KiCad schematic)
At the start: 0 parts

Commit message: Actualizacion estoy cansado jefe :)
Parts:
- added K1, K2: SRA-24VDC-CL, cris:SOT-23-6_L2.9-W1.6-P0.95-LS2.8-BR, symbol Cris:SRA-24VDC-CL
- added U3: LK1802, cris:SOT-23-6_L2.9-W1.6-P0.95-LS2.8-BR, symbol Cris:LK1802
Connections:
- net RLY1_C: now also K2.5
- net RLY1_NC: now also K2.2
- net RLY1_NO: now also K2.1
- net RLY2_C: now also K1.5
- net RLY2_NC: now also K1.2
- net RLY2_NO: now also K1.1
- net RLY_1: now also U3.3 (1B)
- net RLY_2: now also U3.4 (2B)
- new net: K1.4, U3.6 (2C)
- new net GND: K2.4, U3.2 (E)
- new net VCC: K1.3, K2.3, U3.5 (COM)

Commit message: Actualizacion 20 :[
Connections:
- net GND: no longer K2.4
- net at U3.1 (1C): now also K2.4
Changed lines of the file:
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@@
 	(wire
 		(pts
-			(xy 144.78 62.23) (xy 144.78 58.42)
+			(xy 144.78 58.42) (xy 144.78 68.58)
 		)
 		(stroke
@@
 		(pts
 			(xy 187.96 68.58) (xy 209.55 68.58)
+		)
+		(stroke
+			(width 0)
+			(type default)
+		)
+	)
+	(wire
+		(pts
+			(xy 170.18 68.58) (xy 144.78 68.58)
 		)
 		(stroke
@@
 					(unit 1)
 				)
-			)
-		)
-	)
-	(symbol
-		(lib_id "power:GND")
-		(at 144.78 62.23 0)
-		(unit 1)
-		(exclude_from_sim no)
-		(in_bom yes)
-		(on_board yes)
-		(dnp no)
-		(fields_autoplaced yes)
-		(property "Reference" "#PWR033"
-			(at 144.78 68.58 0)
-			(effects
-				(font
-					(size 1.27 1.27)
-				)
-				(hide yes)
-			)
-		)
-		(property "Value" "GND"
-			(at 144.78 67.31 0)
-			(effects
-				(font
-					(size 1.27 1.27)
-				)
-			)
-		)
-		(property "Footprint" ""
-			(at 144.78 62.23 0)
-			(effects
-				(font
-					(size 1.27 1.27)
-				)
-				(hide yes)
-			)
-		)
-		(property "Datasheet" ""
-			(at 144.78 62.23 0)
-			(effects
-				(font
-					(size 1.27 1.27)
-				)
-				(hide yes)
-			)
-		)
-		(property "Description" "Power symbol creates a global label with name \"GND\" , ground"
-			(at 144.78 62.23 0)
-			(effects
-				(font
-					(size 1.27 1.27)
-				)
-				(hide yes)
-			)
-		)
-		(pin "1"
-		)
-		(instances
-			(project ""
-				(path "/3591d221-fcc3-4bcd-9e55-dff6b841bafc/6cae9003-6268-4873-a546-b84fa61fb294/59f81767-a196-4819-bb61-d9fce72f6c5d"
-					(reference "#PWR033")
-					(unit 1)
-				)
