File: KICAD diseño/PLC DISEÑO/PLC DISEÑO.kicad_pcb (KiCad board)
At the start: 2 copper layers, 0 parts

Commit message: Update
Parts:
- added C1: 1u, PCM_Capacitor_SMD_AKL:C_0603_1608Metric, F.Cu at (74.7, 86.7)
- added C2: C_0603, PCM_Capacitor_SMD_AKL:C_0603_1608Metric, F.Cu at (60.1, 86.7)
- added C3: 100pF, PCM_Capacitor_SMD_AKL:C_0603_1608Metric, F.Cu at (60.1, 89.4)
- added C4: 100pF, PCM_Capacitor_SMD_AKL:C_0603_1608Metric, F.Cu at (60.1, 92.1)
- added C5: 22uF, PCM_Capacitor_SMD_AKL:C_0603_1608Metric, F.Cu at (91.3, 87.7)
- added C6: 22uF, PCM_Capacitor_SMD_AKL:C_0603_1608Metric, F.Cu at (91.3, 90.4)
- added C7: ~, Library:C2992406, F.Cu at (70.8, 59.6)
- added J1: Screw_Terminal_2_P5.00mm, TerminalBlock_Phoenix:TerminalBlock_Phoenix_PT-1,5-2-5.0-H_1x02_P5.00mm_Horizontal, F.Cu at (90.0, 108.5)
- added J10: Screw_Terminal_3_P5.00mm, TerminalBlock_Phoenix:TerminalBlock_Phoenix_PT-1,5-3-5.0-H_1x03_P5.00mm_Horizontal, F.Cu at (110.0, 41.2)
- added J11: Screw_Terminal_2_P5.00mm, TerminalBlock_Phoenix:TerminalBlock_Phoenix_PT-1,5-2-5.0-H_1x02_P5.00mm_Horizontal, F.Cu at (39.8, 89.8)
- added J14: Screw_Terminal_6_P5.00mm, TerminalBlock_Phoenix:TerminalBlock_Phoenix_PT-1,5-6-5.0-H_1x06_P5.00mm_Horizontal, F.Cu at (38.2, 41.2)
- added J2: Screw_Terminal_4_P5.00mm, TerminalBlock_Phoenix:TerminalBlock_Phoenix_PT-1,5-4-5.0-H_1x04_P5.00mm_Horizontal, F.Cu at (70.5, 41.2)
- added J3: Screw_Terminal_2_P5.00mm, TerminalBlock_Phoenix:TerminalBlock_Phoenix_PT-1,5-2-5.0-H_1x02_P5.00mm_Horizontal, F.Cu at (74.5, 107.2)
- added J4: Screw_Terminal_2_P5.00mm, TerminalBlock_Phoenix:TerminalBlock_Phoenix_PT-1,5-2-5.0-H_1x02_P5.00mm_Horizontal, F.Cu at (39.8, 56.6)
- added J6: Screw_Terminal_3_P5.00mm, TerminalBlock_Phoenix:TerminalBlock_Phoenix_PT-1,5-3-5.0-H_1x03_P5.00mm_Horizontal, F.Cu at (92.5, 41.0)
- added J7: Screw_Terminal_2_P5.00mm, TerminalBlock_Phoenix:TerminalBlock_Phoenix_PT-1,5-2-5.0-H_1x02_P5.00mm_Horizontal, F.Cu at (39.8, 67.7)
- added J8: Screw_Terminal_2_P5.00mm, TerminalBlock_Phoenix:TerminalBlock_Phoenix_PT-1,5-2-5.0-H_1x02_P5.00mm_Horizontal, F.Cu at (39.8, 78.8)
- added J9: Screw_Terminal_4_P5.00mm, TerminalBlock_Phoenix:TerminalBlock_Phoenix_PT-1,5-4-5.0-H_1x04_P5.00mm_Horizontal, F.Cu at (50.0, 107.8)
- added L1: L_Iron, PCM_Inductor_SMD_AKL:L_Bourns-SRN6028, F.Cu at (66.4, 89.2)
- added R1: R_0603, PCM_Resistor_SMD_AKL:R_0603_1608Metric, F.Cu at (74.6, 89.4)
- added R2: 22k, PCM_Resistor_SMD_AKL:R_0603_1608Metric, F.Cu at (87.1, 87.7)
- added R3: 22k, PCM_Resistor_SMD_AKL:R_0603_1608Metric, F.Cu at (87.1, 90.4)
- added U2: AP63203WU, Package_TO_SOT_SMD:TSOT-23-6, F.Cu at (64.8, 95.6)

Commit message: Actualizacion
Parts:
- added C8: C_0603, PCM_Capacitor_SMD_AKL:C_0603_1608Metric, F.Cu at (99.7, 76.2)
- added D1: SM712, PCM_Package_TO_SOT_SMD_AKL:SOT-23, F.Cu at (99.9, 72.5)
- added D2: DL4007, PCM_Diode_SMD_AKL:D_MELF, F.Cu at (87.4, 78.5)
- added D3: DL4007, PCM_Diode_SMD_AKL:D_MELF, F.Cu at (87.4, 65.4)
- added OC1: LTV-357T, PCM_Package_SO_AKL:SO-4_4.4x3.9mm_P2.54mm, F.Cu at (88.3, 73.0)
- added OC2: LTV-357T, PCM_Package_SO_AKL:SO-4_4.4x3.9mm_P2.54mm, F.Cu at (88.3, 59.9)
- added R4: R_0603, PCM_Resistor_SMD_AKL:R_0603_1608Metric, F.Cu at (93.5, 77.2)
- added R5: R_0603, PCM_Resistor_SMD_AKL:R_0603_1608Metric, F.Cu at (93.5, 80.0)
- added R6: R_0603, PCM_Resistor_SMD_AKL:R_0603_1608Metric, F.Cu at (93.5, 64.1)
- added R7: R_0603, PCM_Resistor_SMD_AKL:R_0603_1608Metric, F.Cu at (93.5, 66.8)
Connections:
- net /BOARD_NIRVARA/RFL1_NC renamed /RFL1_NC
- net /BOARD_NIRVARA/RFL2_NC renamed /RFL2_NC
- C2 pad 2: unconnected-(C2-Pad2) -> GND
- C7 pad 1: unconnected-(C7-VCC-Pad1) -> +3.3V
- C7 pad 2: unconnected-(C7-GND-Pad2) -> Net-(C7-GND)
- C7 pad 3: unconnected-(C7-TXD-Pad3) -> /BOARD_NIRVARA/DRIVER_RS485/UART_IN
- C7 pad 4: unconnected-(C7-RXD-Pad4) -> /BOARD_NIRVARA/DRIVER_RS485/UART_OUT
- C7 pad 5: unconnected-(C7-CON-Pad5) -> /BOARD_NIRVARA/DRIVER_RS485/GPIO control
- C7 pad 8: unconnected-(C7-A-Pad8) -> /BOARD_NIRVARA/RS485-B
- C7 pad 9: (no net) -> /BOARD_NIRVARA/RS485-A

Commit message: Actualizacion estoy cansado jefe :)
Parts:
- added C10: C_0603, PCM_Capacitor_SMD_AKL:C_0603_1608Metric, F.Cu at (106.8, 65.3)
- added C11: C_0603, PCM_Capacitor_SMD_AKL:C_0603_1608Metric, F.Cu at (106.8, 55.1)
- added C12: C_0603, PCM_Capacitor_SMD_AKL:C_0603_1608Metric, F.Cu at (106.8, 57.8)
- added C9: C_0603, PCM_Capacitor_SMD_AKL:C_0603_1608Metric, F.Cu at (106.8, 62.5)
- added D4: DL4007, PCM_Diode_SMD_AKL:D_MELF, F.Cu at (117.2, 87.3)
- added D5: DL4007, PCM_Diode_SMD_AKL:D_MELF, F.Cu at (117.2, 74.1)
- added D7: SMF24A, PCM_Diode_SMD_AKL:D_SOD-123F, F.Cu at (107.5, 51.7)
- added K1: SRA-24VDC-CL, cris:SOT-23-6_L2.9-W1.6-P0.95-LS2.8-BR, F.Cu at (108.8, 67.9)
- added K2: SRA-24VDC-CL, cris:SOT-23-6_L2.9-W1.6-P0.95-LS2.8-BR, F.Cu at (108.8, 72.5)
- added OC3: LTV-357T, PCM_Package_SO_AKL:SO-4_4.4x3.9mm_P2.54mm, F.Cu at (118.1, 81.8)
- added OC4: LTV-357T, PCM_Package_SO_AKL:SO-4_4.4x3.9mm_P2.54mm, F.Cu at (118.1, 68.6)
- added R10: R_0603, PCM_Resistor_SMD_AKL:R_0603_1608Metric, F.Cu at (123.3, 72.8)
- added R11: R_0603, PCM_Resistor_SMD_AKL:R_0603_1608Metric, F.Cu at (123.3, 75.5)
- added R12: R_0603, PCM_Resistor_SMD_AKL:R_0603_1608Metric, F.Cu at (102.6, 62.5)
- added R13: R_0603, PCM_Resistor_SMD_AKL:R_0603_1608Metric, F.Cu at (102.6, 65.3)
- added R14: R_0603, PCM_Resistor_SMD_AKL:R_0603_1608Metric, F.Cu at (102.6, 68.0)
- added R15: R_0603, PCM_Resistor_SMD_AKL:R_0603_1608Metric, F.Cu at (102.6, 51.0)
- added R16: R_0603, PCM_Resistor_SMD_AKL:R_0603_1608Metric, F.Cu at (102.6, 53.7)
- added R17: R_0603, PCM_Resistor_SMD_AKL:R_0603_1608Metric, F.Cu at (102.6, 56.4)
- added R18: R_0603, PCM_Resistor_SMD_AKL:R_0603_1608Metric, F.Cu at (113.0, 62.5)
- added R8: R_0603, PCM_Resistor_SMD_AKL:R_0603_1608Metric, F.Cu at (123.3, 86.0)
- added R9: R_0603, PCM_Resistor_SMD_AKL:R_0603_1608Metric, F.Cu at (123.3, 88.7)
- added U1: ESP32-S3-WROOM-1, ESP32-S3-WROM-1:ESP32-S3-WROOM-1, F.Cu at (125.5, 103.5)
- added U3: LK1802, cris:SOT-23-6_L2.9-W1.6-P0.95-LS2.8-BR, F.Cu at (108.8, 77.1)
- moved C7 13.0 mm to (70.0, 46.6)
- moved C4 11.4 mm to (63.4, 81.2)
- moved R1 11.4 mm to (77.9, 78.5)
- moved C1 11.4 mm to (78.0, 75.7)
- moved C2 11.4 mm to (63.4, 75.7)
- moved C3 11.4 mm to (63.4, 78.5)
- moved L1 11.4 mm to (69.7, 78.3)
- moved U2 11.4 mm to (68.1, 84.7)
- moved R2 10.9 mm to (76.8, 84.0)
- moved R3 10.9 mm to (76.8, 86.7)
- moved C5 10.9 mm to (81.0, 84.0)
- moved C6 10.9 mm to (81.0, 86.8)
- moved J1 1.25 mm to (89.2, 107.5)
- moved J3 0.50 mm to (74.5, 107.8)
Connections:
- net /BOARD_NIRVARA/INPUT_NPN/NPN_input renamed /BOARD_NIRVARA/INPUT_NPN/NPN_input_1
- net /BOARD_NIRVARA/INPUT_PNP/PNP_input renamed /BOARD_NIRVARA/INPUT_PNP/PNP_input_1
- D2 pad 2: /BOARD_NIRVARA/NPN_IN_1 -> GND
- D3 pad 2: /BOARD_NIRVARA/PNP_IN_2 -> GND
- OC1 pad 2: /BOARD_NIRVARA/NPN_IN_1 -> GND
- OC2 pad 2: /BOARD_NIRVARA/PNP_IN_2 -> GND
- R4 pad 1: /BOARD_NIRVARA/NPN_IN_2 -> /BOARD_NIRVARA/NPN_IN_1

Commit message: Actualizacion 20 :[
Parts:
- added C13: C_0603, PCM_Capacitor_SMD_AKL:C_0603_1608Metric, F.Cu at (96.5, 92.0)
- added C14: C_0603, PCM_Capacitor_SMD_AKL:C_0603_1608Metric, F.Cu at (90.1, 89.7)
- added D8: DL4007, PCM_Diode_SMD_AKL:D_MELF, F.Cu at (81.9, 91.8)
- added D9: DL4007, PCM_Diode_SMD_AKL:D_MELF, F.Cu at (81.9, 97.0)
- added J5: Screw_Terminal_4_P5.00mm, TerminalBlock_Phoenix:TerminalBlock_Phoenix_PT-1,5-4-5.0-H_1x04_P5.00mm_Horizontal, F.Cu at (93.2, 107.2)
- added OC5: LTV-357T, PCM_Package_SO_AKL:SO-4_4.4x3.9mm_P2.54mm, F.Cu at (64.9, 92.5)
- added OC6: LTV-357T, PCM_Package_SO_AKL:SO-4_4.4x3.9mm_P2.54mm, F.Cu at (64.9, 98.2)
- added R19: R_0603, PCM_Resistor_SMD_AKL:R_0603_1608Metric, F.Cu at (96.4, 94.7)
- added R20: R_0603, PCM_Resistor_SMD_AKL:R_0603_1608Metric, F.Cu at (96.4, 97.4)
- added R21: R_0603, PCM_Resistor_SMD_AKL:R_0603_1608Metric, F.Cu at (90.0, 92.5)
- added R22: R_0603, PCM_Resistor_SMD_AKL:R_0603_1608Metric, F.Cu at (71.9, 91.0)
- added R23: R_0603, PCM_Resistor_SMD_AKL:R_0603_1608Metric, F.Cu at (71.9, 93.7)
- added R24: R_0603, PCM_Resistor_SMD_AKL:R_0603_1608Metric, F.Cu at (71.9, 96.5)
- added R25: R_0603, PCM_Resistor_SMD_AKL:R_0603_1608Metric, F.Cu at (71.9, 99.2)
- moved C5 10.9 mm to (78.0, 73.5)
- moved C6 10.9 mm to (78.0, 76.2)
- moved J1 9.76 mm to (79.5, 108.0)
- moved J3 9.33 mm to (65.2, 109.0)
- moved J9 9.03 mm to (41.0, 108.5)
- moved C1 6.23 mm to (72.1, 73.9)
- moved L1 6.23 mm to (63.8, 76.5)
- moved R2 6.23 mm to (70.8, 82.2)
- moved R3 6.23 mm to (70.8, 84.9)
- moved R1 6.23 mm to (72.0, 76.6)
- moved C2 6.23 mm to (57.4, 73.9)
- moved C3 6.23 mm to (57.4, 76.6)
- moved U2 6.23 mm to (62.2, 82.9)
- moved C4 6.23 mm to (57.4, 79.3)
Connections:
- J14 pad 1: /RFL1_NC -> /BOARD_NIRVARA/RLY1_NC
- J14 pad 4: /RFL2_NC -> /BOARD_NIRVARA/RLY2_NC
- U1 pad 12: unconnected-(U1-GPIO8/TOUCH8/ADC1_CH7/SUBSPICS1-Pad12) -> /BOARD_NIRVARA/Modulo_out_420/SDA
- U1 pad 15: unconnected-(U1-GPIO3/TOUCH3/ADC1_CH2-Pad15) -> /BOARD_NIRVARA/INPUT_PNP/PNP_input_1
- U1 pad 16: unconnected-(U1-GPIO46-Pad16) -> /BOARD_NIRVARA/Modulo_in/input_2
- U1 pad 17: unconnected-(U1-GPIO9/TOUCH9/ADC1_CH8/FSPIHD/SUBSPIHD-Pad17) -> /BOARD_NIRVARA/Modulo_010/SDA
- U1 pad 18: unconnected-(U1-GPIO10/TOUCH10/ADC1_CH9/FSPICS0/FSPIIO4/SUBSPICS0-Pad18) -> /BOARD_NIRVARA/Modulo_010/SCLK
- U1 pad 19: unconnected-(U1-GPIO11/TOUCH11/ADC2_CH0/FSPID/FSPIIO5/SUBSPID-Pad19) -> /BOARD_NIRVARA/34_v/0_32Vin
- U1 pad 26: unconnected-(U1-GPIO45-Pad26) -> /BOARD_NIRVARA/Modulo_in/input_1
- U1 pad 27: unconnected-(U1-GPIO0/BOOT-Pad27) -> /BOARD_NIRVARA/420_IN/420_in
- U1 pad 38: unconnected-(U1-GPIO2/TOUCH2/ADC1_CH1-Pad38) -> /BOARD_NIRVARA/INPUT_NPN/NPN_input_2
- U1 pad 39: unconnected-(U1-GPIO1/TOUCH1/ADC1_CH0-Pad39) -> /BOARD_NIRVARA/INPUT_NPN/NPN_input_1
- U1 pad 4: unconnected-(U1-GPIO4/TOUCH4/ADC1_CH3-Pad4) -> /BOARD_NIRVARA/INPUT_PNP/PNP_input_2
- U1 pad 5: unconnected-(U1-GPIO5/TOUCH5/ADC1_CH4-Pad5) -> /BOARD_NIRVARA/Realy/RLY_1
- U1 pad 6: unconnected-(U1-GPIO6/TOUCH6/ADC1_CH5-Pad6) -> /BOARD_NIRVARA/Realy/RLY_2
- U1 pad 7: unconnected-(U1-GPIO7/TOUCH7/ADC1_CH6-Pad7) -> /BOARD_NIRVARA/Modulo_out_420/ASLK

Commit message: uptade
Parts:
- added C15: C_0603, PCM_Capacitor_SMD_AKL:C_0603_1608Metric, F.Cu at (122.4, 56.8)
- added R26: R_0603, PCM_Resistor_SMD_AKL:R_0603_1608Metric, F.Cu at (122.3, 59.6)
- added R27: R_0603, PCM_Resistor_SMD_AKL:R_0603_1608Metric, F.Cu at (122.3, 62.3)
- added R28: R_0603, PCM_Resistor_SMD_AKL:R_0603_1608Metric, F.Cu at (128.7, 56.8)
- added R29: R_0603, PCM_Resistor_SMD_AKL:R_0603_1608Metric, F.Cu at (128.7, 59.6)
- added R30: R_0603, PCM_Resistor_SMD_AKL:R_0603_1608Metric, F.Cu at (128.7, 64.3)
- added R31: R_0603, PCM_Resistor_SMD_AKL:R_0603_1608Metric, F.Cu at (128.7, 67.0)
Connections:
- C14 pad 1: /BOARD_NIRVARA/420_IN/420_in -> /BOARD_NIRVARA/A420_IN1
- K2 pad 4: GND -> Net-(U3-1C)
- R21 pad 1: /BOARD_NIRVARA/420_IN/420_in -> /BOARD_NIRVARA/A420_IN1
- U1 pad 10: unconnected-(U1-GPIO17/U1TXD/ADC2_CH6-Pad10) -> /BOARD_NIRVARA/0.10Vin/0-10V
- U1 pad 11: unconnected-(U1-GPIO18/U1RXD/ADC2_CH7/CLK_OUT3-Pad11) -> /BOARD_NIRVARA/34_v/0_32Vin
- U1 pad 12: /BOARD_NIRVARA/Modulo_out_420/SDA -> /BOARD_NIRVARA/INPUT_PNP/PNP_input_2
- U1 pad 13: unconnected-(U1-GPIO19/U1RTS/ADC2_CH8/CLK_OUT2/USB_D--Pad13) -> /BOARD_NIRVARA/Realy/RLY_2
- U1 pad 14: unconnected-(U1-GPIO20/U1CTS/ADC2_CH9/CLK_OUT1/USB_D+-Pad14) -> /BOARD_NIRVARA/Realy/RLY_1
- U1 pad 15: /BOARD_NIRVARA/INPUT_PNP/PNP_input_1 -> /BOARD_NIRVARA/Out_PNP/PNP-1
- U1 pad 16: /BOARD_NIRVARA/Modulo_in/input_2 -> unconnected-(U1-GPIO46-Pad16)
- U1 pad 19: /BOARD_NIRVARA/34_v/0_32Vin -> /BOARD_NIRVARA/Modulo_out_420/ASLK
- U1 pad 20: unconnected-(U1-GPIO12/TOUCH12/ADC2_CH1/FSPICLK/FSPIIO6/SUBSPICLK-Pad20) -> /BOARD_NIRVARA/Modulo_out_420/SDA
- U1 pad 21: unconnected-(U1-GPIO13/TOUCH13/ADC2_CH2/FSPIQ/FSPIIO7/SUBSPIQ-Pad21) -> /BOARD_NIRVARA/DRIVER_RS485/UART_IN
- U1 pad 22: unconnected-(U1-GPIO14/TOUCH14/ADC2_CH3/FSPIWP/FSPIDQS/SUBSPIWP-Pad22) -> /BOARD_NIRVARA/DRIVER_RS485/UART_OUT
- U1 pad 23: unconnected-(U1-GPIO21-Pad23) -> /BOARD_NIRVARA/A420_IN1
- U1 pad 26: /BOARD_NIRVARA/Modulo_in/input_1 -> unconnected-(U1-GPIO45-Pad26)
- U1 pad 27: /BOARD_NIRVARA/420_IN/420_in -> unconnected-(U1-GPIO0/BOOT-Pad27)
- U1 pad 36: /BOARD_NIRVARA/DRIVER_RS485/UART_OUT -> /BOARD_NIRVARA/Modulo_in/input_2
- U1 pad 37: /BOARD_NIRVARA/DRIVER_RS485/UART_IN -> /BOARD_NIRVARA/Modulo_in/input_1
- U1 pad 38: /BOARD_NIRVARA/INPUT_NPN/NPN_input_2 -> /BOARD_NIRVARA/Out_NPN/NPN-2
- U1 pad 39: /BOARD_NIRVARA/INPUT_NPN/NPN_input_1 -> /BOARD_NIRVARA/Out_NPN/NPN-1
- U1 pad 4: /BOARD_NIRVARA/INPUT_PNP/PNP_input_2 -> /BOARD_NIRVARA/Out_PNP/PNP-2
- U1 pad 5: /BOARD_NIRVARA/Realy/RLY_1 -> /BOARD_NIRVARA/INPUT_NPN/NPN_input_1
- U1 pad 6: /BOARD_NIRVARA/Realy/RLY_2 -> /BOARD_NIRVARA/INPUT_NPN/NPN_input_2
- U1 pad 7: /BOARD_NIRVARA/Modulo_out_420/ASLK -> /BOARD_NIRVARA/INPUT_PNP/PNP_input_1
- U3 pad 1: unconnected-(U3-1C-Pad1) -> Net-(U3-1C)

Commit message: update
Parts:
- moved C10 225.0 mm to (232.0, 252.2)
- moved C9 225.0 mm to (232.0, 249.5)
- moved R12 225.0 mm to (227.7, 249.5)
- moved R13 225.0 mm to (227.7, 252.2)
- moved R14 225.0 mm to (227.7, 254.9)
- moved D3 204.0 mm to (170.7, 251.6)
- moved R6 204.0 mm to (176.8, 250.3)
- moved R7 204.0 mm to (176.8, 253.0)
- moved OC4 194.1 mm to (193.4, 247.6)
- moved R10 194.1 mm to (198.6, 251.8)
- moved R11 194.1 mm to (198.6, 254.5)
- moved D5 194.1 mm to (192.5, 253.1)
- moved R19 192.2 mm to (248.7, 212.0)
- moved R20 192.2 mm to (248.7, 214.8)
- moved C13 192.2 mm to (248.8, 209.3)
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